Commit message: added moveable fingers to xacro

File: spotarm_assembly_description/urdf/spotarm_assembly.xacro (robot description, xacro)
@@ -145,4 +145,37 @@
   </collision>
 </link>
+<link name="gripper_right_finger">
+  <visual>
+    <origin xyz="0 0 0" rpy="0 0 0"/>
+    <geometry>
+      <box size="0.005 0.02 0.0192"/>
+    </geometry>
+    <material name="silver"/>
+  </visual>
+</link>
+<link name="gripper_left_finger">
+  <visual>
+    <origin xyz="0 0 0" rpy="0 0 0"/>
+    <geometry>
+      <box size="0.005 0.02 0.0192"/>
+    </geometry>
+    <material name="silver"/>
+  </visual>
+</link>
+<joint name="gripper_right_finger_joint" type="prismatic">
+  <parent link="gripper_1"/>
+  <child link="gripper_right_finger"/>
+  <origin xyz="-0.021 -0.0965 -0.0170" rpy="0.175 0 0"/>
+  <axis xyz="1 0 0"/>
+  <limit lower="0.0" upper="0.0185" effort="10.0" velocity="0.02"/>
+</joint>
+<joint name="gripper_left_finger_joint" type="prismatic">
+  <parent link="gripper_1"/>
+  <child link="gripper_left_finger"/>
+  <origin xyz="0.021 -0.0965 -0.0170" rpy="0.175 0 0"/>
+  <axis xyz="-1 0 0"/>
+  <mimic joint="gripper_right_finger_joint"/>
+  <limit lower="0.0" upper="0.0185" effort="10.0" velocity="0.02"/>
+</joint>
 <joint name="Revolute1" type="revolute">
   <origin xyz="0.02835 -0.011972 0.033179" rpy="0 0 0"/>
@@ -171,5 +204,5 @@
 </joint>
 <joint name="Revolute5" type="continuous">
-  <origin xyz="0.0705 -0.143933 0.0" rpy="0 0 0"/>
+  <origin xyz="0.0705 -0.143933 0.0" rpy="-0.175 0 0"/>
   <parent link="link_5_1"/>
   <child link="link_6_1"/>
