Commit message: created new moveit config with updated cad model

File: robot_moveit_config/config/spotarm_assembly.ros2_control.xacro (robot description, xacro)
@@ -8,43 +8,43 @@
                 <plugin>mock_components/GenericSystem</plugin>
             </hardware>
-            <joint name="Revolute1">
+            <joint name="Revolute 1">
                 <command_interface name="position"/>
                 <state_interface name="position">
-                  <param name="initial_value">${initial_positions['Revolute1']}</param>
+                  <param name="initial_value">${initial_positions['Revolute 1']}</param>
                 </state_interface>
                 <state_interface name="velocity"/>
             </joint>
-            <joint name="Revolute2">
+            <joint name="Revolute 2">
                 <command_interface name="position"/>
                 <state_interface name="position">
-                  <param name="initial_value">${initial_positions['Revolute2']}</param>
+                  <param name="initial_value">${initial_positions['Revolute 2']}</param>
                 </state_interface>
                 <state_interface name="velocity"/>
             </joint>
-            <joint name="Revolute3">
+            <joint name="Revolute 3">
                 <command_interface name="position"/>
                 <state_interface name="position">
-                  <param name="initial_value">${initial_positions['Revolute3']}</param>
+                  <param name="initial_value">${initial_positions['Revolute 3']}</param>
                 </state_interface>
                 <state_interface name="velocity"/>
             </joint>
-            <joint name="Revolute4">
+            <joint name="Revolute 4">
                 <command_interface name="position"/>
                 <state_interface name="position">
-                  <param name="initial_value">${initial_positions['Revolute4']}</param>
+                  <param name="initial_value">${initial_positions['Revolute 4']}</param>
                 </state_interface>
                 <state_interface name="velocity"/>
             </joint>
-            <joint name="Revolute5">
+            <joint name="Revolute 5">
                 <command_interface name="position"/>
                 <state_interface name="position">
-                  <param name="initial_value">${initial_positions['Revolute5']}</param>
+                  <param name="initial_value">${initial_positions['Revolute 5']}</param>
                 </state_interface>
                 <state_interface name="velocity"/>
             </joint>
-            <joint name="Revolute6">
+            <joint name="Revolute 6">
                 <command_interface name="position"/>
                 <state_interface name="position">
-                  <param name="initial_value">${initial_positions['Revolute6']}</param>
+                  <param name="initial_value">${initial_positions['Revolute 6']}</param>
                 </state_interface>
                 <state_interface name="velocity"/>

File: spotarm_assembly_description/urdf/spotarm_assembly.xacro (robot description, xacro)
@@ -4,5 +4,4 @@
 <xacro:include filename="$(find spotarm_assembly_description)/urdf/spotarm_assembly.trans" />
 <xacro:include filename="$(find spotarm_assembly_description)/urdf/spotarm_assembly.gazebo" />
-<xacro:include filename="spotarm_assembly.ros2_control.xacro"/>
 <link name="base_link">
   <inertial>
@@ -25,5 +24,5 @@
   </collision>
 </link>
-<link name="link_2">
+<link name="link_2_1">
   <inertial>
     <origin xyz="-0.012527874109626764 -0.0005474727478518779 0.05618235883344737" rpy="0 0 0"/>
@@ -34,5 +33,5 @@
     <origin xyz="-0.02835 0.011972 -0.033179" rpy="0 0 0"/>
     <geometry>
-      <mesh filename="file://$(find spotarm_assembly_description)/meshes/Joint_2_Component_v2_1.stl" scale="0.001 0.001 0.001"/>
+      <mesh filename="file://$(find spotarm_assembly_description)/meshes/link_2_1.stl" scale="0.001 0.001 0.001"/>
     </geometry>
     <material name="silver"/>
@@ -41,9 +40,9 @@
     <origin xyz="-0.02835 0.011972 -0.033179" rpy="0 0 0"/>
     <geometry>
-      <mesh filename="file://$(find spotarm_assembly_description)/meshes/Joint_2_Component_v2_1.stl" scale="0.001 0.001 0.001"/>
+      <mesh filename="file://$(find spotarm_assembly_description)/meshes/link_2_1.stl" scale="0.001 0.001 0.001"/>
     </geometry>
   </collision>
 </link>
-<link name="link_3">
+<link name="link_3_1">
   <inertial>
     <origin xyz="-0.0023570645830831988 -0.2070530002719938 0.00014934365865988675" rpy="0 0 0"/>
@@ -54,5 +53,5 @@
     <origin xyz="-0.074358 0.011972 -0.109385" rpy="0 0 0"/>
     <geometry>
-      <mesh filename="file://$(find spotarm_assembly_description)/meshes/Joint_3_Component_v2_1.stl" scale="0.001 0.001 0.001"/>
+      <mesh filename="file://$(find spotarm_assembly_description)/meshes/link_3_1.stl" scale="0.001 0.001 0.001"/>
     </geometry>
     <material name="silver"/>
@@ -61,9 +60,9 @@
     <origin xyz="-0.074358 0.011972 -0.109385" rpy="0 0 0"/>
     <geometry>
-      <mesh filename="file://$(find spotarm_assembly_description)/meshes/Joint_3_Component_v2_1.stl" scale="0.001 0.001 0.001"/>
+      <mesh filename="file://$(find spotarm_assembly_description)/meshes/link_3_1.stl" scale="0.001 0.001 0.001"/>
     </geometry>
   </collision>
 </link>
-<link name="link_4">
+<link name="link_4_1">
   <inertial>
     <origin xyz="-0.014428046075399614 -0.08611675195042084 -0.0016741934805408476" rpy="0 0 0"/>
@@ -74,5 +73,5 @@
     <origin xyz="-0.001798 0.325662 -0.109385" rpy="0 0 0"/>
     <geometry>
-      <mesh filename="file://$(find spotarm_assembly_description)/meshes/Joint_4_Component_v2_1.stl" scale="0.001 0.001 0.001"/>
+      <mesh filename="file://$(find spotarm_assembly_description)/meshes/link_4_1.stl" scale="0.001 0.001 0.001"/>
     </geometry>
     <material name="silver"/>
@@ -81,9 +80,9 @@
     <origin xyz="-0.001798 0.325662 -0.109385" rpy="0 0 0"/>
     <geometry>
-      <mesh filename="file://$(find spotarm_assembly_description)/meshes/Joint_4_Component_v2_1.stl" scale="0.001 0.001 0.001"/>
+      <mesh filename="file://$(find spotarm_assembly_description)/meshes/link_4_1.stl" scale="0.001 0.001 0.001"/>
     </geometry>
   </collision>
 </link>
-<link name="link_5">
+<link name="link_5_1">
   <inertial>
     <origin xyz="-8.830559206677441e-05 -0.10284977811786078 -0.00047877688390274287" rpy="0 0 0"/>
@@ -94,5 +93,5 @@
     <origin xyz="0.010663 0.537462 -0.109385" rpy="0 0 0"/>
     <geometry>
-      <mesh filename="file://$(find spotarm_assembly_description)/meshes/Joint_5_Component_v2_1.stl" scale="0.001 0.001 0.001"/>
+      <mesh filename="file://$(find spotarm_assembly_description)/meshes/link_5_1.stl" scale="0.001 0.001 0.001"/>
     </geometry>
     <material name="silver"/>
@@ -101,123 +100,83 @@
     <origin xyz="0.010663 0.537462 -0.109385" rpy="0 0 0"/>
     <geometry>
-      <mesh filename="file://$(find spotarm_assembly_description)/meshes/Joint_5_Component_v2_1.stl" scale="0.001 0.001 0.001"/>
+      <mesh filename="file://$(find spotarm_assembly_description)/meshes/link_5_1.stl" scale="0.001 0.001 0.001"/>
     </geometry>
   </collision>
 </link>
-<link name="link_6_fake">
+<link name="link_6_1">
   <inertial>
-    <origin xyz="0.011 -0.09 0" rpy="0 0 0"/>
-    <mass value="0.2"/>
-    <inertia ixx="1.3333333333333334e-05" iyy="4.8333333333333334e-05" izz="4.8333333333333334e-05" ixy="0.0" iyz="0.0" ixz="0.0"/>
+    <origin xyz="0.012673058332606776 -0.0664264989047959 -0.014305380960634592" rpy="0 0 0"/>
+    <mass value="4.625546361310207"/>
+    <inertia ixx="0.014614" iyy="0.003535" izz="0.014333" ixy="0.000114" iyz="-0.00222" ixz="3.5e-05"/>
   </inertial>
   <visual>
-    <origin xyz="0.011 -0.09 0" rpy="0 0 0"/>
+    <origin xyz="-0.059837 0.681395 -0.109385" rpy="0 0 0"/>
     <geometry>
-      <box size="0.02 0.2 0.02"/>
+      <mesh filename="file://$(find spotarm_assembly_description)/meshes/link_6_1.stl" scale="0.001 0.001 0.001"/>
     </geometry>
     <material name="silver"/>
   </visual>
   <collision>
-    <origin xyz="0.011 -0.09 0" rpy="0 0 0"/>
+    <origin xyz="-0.059837 0.681395 -0.109385" rpy="0 0 0"/>
     <geometry>
-      <box size="0.02 0.2 0.02"/>
+      <mesh filename="file://$(find spotarm_assembly_description)/meshes/link_6_1.stl" scale="0.001 0.001 0.001"/>
     </geometry>
   </collision>
 </link>
-<link name="link_7_fake">
+<link name="gripper_1">
   <inertial>
-    <origin xyz="0 -0.1 0" rpy="0 0 0"/>
-    <mass value="0.2"/>
-    <inertia ixx="1.3333333333333334e-05" iyy="4.8333333333333334e-05" izz="4.8333333333333334e-05" ixy="0.0" iyz="0.0" ixz="0.0"/>
+    <origin xyz="-0.0007404974490983068 -0.036613651652765644 -0.008144219074578796" rpy="0 0 0"/>
+    <mass value="2.203716226137548"/>
+    <inertia ixx="0.001814" iyy="0.001382" izz="0.001879" ixy="-3.5e-05" iyz="-0.000177" ixz="-3.9e-05"/>
   </inertial>
   <visual>
-    <origin xyz="0 -0.05 0" rpy="0 0 0"/>
+    <origin xyz="-0.072537 0.836158 -0.082096" rpy="0 0 0"/>
     <geometry>
-      <box size="0.02 0.1 0.02"/>
+      <mesh filename="file://$(find spotarm_assembly_description)/meshes/gripper_1.stl" scale="0.001 0.001 0.001"/>
     </geometry>
     <material name="silver"/>
   </visual>
   <collision>
-    <origin xyz="0 -0.1 0" rpy="0 0 0"/>
+    <origin xyz="-0.072537 0.836158 -0.082096" rpy="0 0 0"/>
     <geometry>
-      <box size="0.02 0.2 0.02"/>
+      <mesh filename="file://$(find spotarm_assembly_description)/meshes/gripper_1.stl" scale="0.001 0.001 0.001"/>
     </geometry>
   </collision>
 </link>
-<link name="fake_gripper">
-  <inertial>
-    <origin xyz="0 -0.04 0" rpy="0 0 0"/>
-    <mass value="0.05"/>
-    <inertia ixx="3.333333333333334e-05" iyy="1.3333333333333334e-05" izz="3.333333333333334e-05" ixy="0.0" iyz="0.0" ixz="0.0"/>
-  </inertial>
-  <visual>
-    <origin xyz="0 -0.01 0" rpy="0 0 0"/>
-    <geometry>
-      <box size="0.04 0.02 0.04"/>
-    </geometry>
-    <material name="silver"/>
-  </visual>
-  <visual>
-    <origin xyz="0.015 -0.05 0" rpy="0 0 0"/>
-    <geometry>
-      <box size="0.01 0.06 0.01"/>
-    </geometry>
-    <material name="silver"/>
-  </visual>
-  <visual>
-    <origin xyz="-0.015 -0.05 0" rpy="0 0 0"/>
-    <geometry>
-      <box size="0.01 0.06 0.01"/>
-    </geometry>
-    <material name="silver"/>
-  </visual>
-  <collision>
-    <origin xyz="0 -0.04 0" rpy="0 0 0"/>
-    <geometry>
-      <box size="0.04 0.08 0.04"/>
-    </geometry>
-  </collision>
-</link>
-<joint name="Revolute1" type="revolute">
+<joint name="Revolute 1" type="continuous">
   <origin xyz="0.02835 -0.011972 0.033179" rpy="0 0 0"/>
   <parent link="base_link"/>
-  <child link="link_2"/>
+  <child link="link_2_1"/>
   <axis xyz="-0.0 0.0 1.0"/>
-  <limit lower="-0.436" upper="2.13" effort="30.0" velocity="1.0"/>
 </joint>
-<joint name="Revolute2" type="continuous">
+<joint name="Revolute 2" type="continuous">
   <origin xyz="0.046008 0.0 0.076206" rpy="0 0 0"/>
-  <parent link="link_2"/>
-  <child link="link_3"/>
+  <parent link="link_2_1"/>
+  <child link="link_3_1"/>
   <axis xyz="1.0 -0.0 -0.0"/>
 </joint>
-<joint name="Revolute3" type="continuous">
+<joint name="Revolute 3" type="continuous">
   <origin xyz="-0.07256 -0.31369 0.0" rpy="0 0 0"/>
-  <parent link="link_3"/>
-  <child link="link_4"/>
+  <parent link="link_3_1"/>
+  <child link="link_4_1"/>
   <axis xyz="-1.0 0.0 0.0"/>
 </joint>
-<joint name="Revolute4" type="continuous">
+<joint name="Revolute 4" type="continuous">
   <origin xyz="-0.012461 -0.2118 0.0" rpy="0 0 0"/>
-  <parent link="link_4"/>
-  <child link="link_5"/>
+  <parent link="link_4_1"/>
+  <child link="link_5_1"/>
   <axis xyz="-0.0 -1.0 0.0"/>
 </joint>
-<joint name="Revolute5" type="continuous">
-  <origin xyz="0.07 -0.144 0" rpy="0 0 0"/>
-  <parent link="link_5"/>
-  <child link="link_6_fake"/>
-  <axis xyz="1.0 0.0 0.0"/>
+<joint name="Revolute 5" type="continuous">
+  <origin xyz="0.0705 -0.143933 0.0" rpy="0 0 0"/>
+  <parent link="link_5_1"/>
+  <child link="link_6_1"/>
+  <axis xyz="1.0 -0.0 -0.0"/>
 </joint>
-<joint name="Revolute6" type="continuous">
-  <origin xyz="0.011 -0.19 0" rpy="0 0 0"/>
-  <parent link="link_6_fake"/>
-  <child link="link_7_fake"/>
-  <axis xyz="0.0 1.0 0.0"/>
-</joint>
-<joint name="fake_gripper_fixed" type="fixed">
-  <origin xyz="0 -0.1 0" rpy="0 0 0"/>
-  <parent link="link_7_fake"/>
-  <child link="fake_gripper"/>
+<joint name="Revolute 6" type="continuous">
+  <origin xyz="0.0127 -0.154763 -0.027289" rpy="0 0 0"/>
+  <parent link="link_6_1"/>
+  <child link="gripper_1"/>
+  <axis xyz="0.0 0.984808 0.173648"/>
 </joint>
 </robot>

Commit message: new cad model now visible in rviz

File: robot_moveit_config/config/spotarm_assembly.ros2_control.xacro (robot description, xacro)
@@ -8,43 +8,43 @@
                 <plugin>mock_components/GenericSystem</plugin>
             </hardware>
-            <joint name="Revolute 1">
+            <joint name="Revolute1">
                 <command_interface name="position"/>
                 <state_interface name="position">
-                  <param name="initial_value">${initial_positions['Revolute 1']}</param>
+                  <param name="initial_value">${initial_positions['Revolute1']}</param>
                 </state_interface>
                 <state_interface name="velocity"/>
             </joint>
-            <joint name="Revolute 2">
+            <joint name="Revolute2">
                 <command_interface name="position"/>
                 <state_interface name="position">
-                  <param name="initial_value">${initial_positions['Revolute 2']}</param>
+                  <param name="initial_value">${initial_positions['Revolute2']}</param>
                 </state_interface>
                 <state_interface name="velocity"/>
             </joint>
-            <joint name="Revolute 3">
+            <joint name="Revolute3">
                 <command_interface name="position"/>
                 <state_interface name="position">
-                  <param name="initial_value">${initial_positions['Revolute 3']}</param>
+                  <param name="initial_value">${initial_positions['Revolute3']}</param>
                 </state_interface>
                 <state_interface name="velocity"/>
             </joint>
-            <joint name="Revolute 4">
+            <joint name="Revolute4">
                 <command_interface name="position"/>
                 <state_interface name="position">
-                  <param name="initial_value">${initial_positions['Revolute 4']}</param>
+                  <param name="initial_value">${initial_positions['Revolute4']}</param>
                 </state_interface>
                 <state_interface name="velocity"/>
             </joint>
-            <joint name="Revolute 5">
+            <joint name="Revolute5">
                 <command_interface name="position"/>
                 <state_interface name="position">
-                  <param name="initial_value">${initial_positions['Revolute 5']}</param>
+                  <param name="initial_value">${initial_positions['Revolute5']}</param>
                 </state_interface>
                 <state_interface name="velocity"/>
             </joint>
-            <joint name="Revolute 6">
+            <joint name="Revolute6">
                 <command_interface name="position"/>
                 <state_interface name="position">
-                  <param name="initial_value">${initial_positions['Revolute 6']}</param>
+                  <param name="initial_value">${initial_positions['Revolute6']}</param>
                 </state_interface>
                 <state_interface name="velocity"/>

File: spotarm_assembly_description/urdf/spotarm_assembly.xacro (robot description, xacro)
@@ -4,4 +4,5 @@
 <xacro:include filename="$(find spotarm_assembly_description)/urdf/spotarm_assembly.trans" />
 <xacro:include filename="$(find spotarm_assembly_description)/urdf/spotarm_assembly.gazebo" />
+<xacro:include filename="spotarm_assembly.ros2_control.xacro"/>
 <link name="base_link">
   <inertial>
@@ -144,11 +145,12 @@
   </collision>
 </link>
-<joint name="Revolute 1" type="continuous">
+<joint name="Revolute1" type="revolute">
   <origin xyz="0.02835 -0.011972 0.033179" rpy="0 0 0"/>
   <parent link="base_link"/>
   <child link="link_2_1"/>
   <axis xyz="-0.0 0.0 1.0"/>
+  <limit lower="-0.436" upper="2.13" effort="30.0" velocity="1.0"/>
 </joint>
-<joint name="Revolute 2" type="continuous">
+<joint name="Revolute2" type="continuous">
   <origin xyz="0.046008 0.0 0.076206" rpy="0 0 0"/>
   <parent link="link_2_1"/>
@@ -156,5 +158,5 @@
   <axis xyz="1.0 -0.0 -0.0"/>
 </joint>
-<joint name="Revolute 3" type="continuous">
+<joint name="Revolute3" type="continuous">
   <origin xyz="-0.07256 -0.31369 0.0" rpy="0 0 0"/>
   <parent link="link_3_1"/>
@@ -162,5 +164,5 @@
   <axis xyz="-1.0 0.0 0.0"/>
 </joint>
-<joint name="Revolute 4" type="continuous">
+<joint name="Revolute4" type="continuous">
   <origin xyz="-0.012461 -0.2118 0.0" rpy="0 0 0"/>
   <parent link="link_4_1"/>
@@ -168,5 +170,5 @@
   <axis xyz="-0.0 -1.0 0.0"/>
 </joint>
-<joint name="Revolute 5" type="continuous">
+<joint name="Revolute5" type="continuous">
   <origin xyz="0.0705 -0.143933 0.0" rpy="0 0 0"/>
   <parent link="link_5_1"/>
@@ -174,5 +176,5 @@
   <axis xyz="1.0 -0.0 -0.0"/>
 </joint>
-<joint name="Revolute 6" type="continuous">
+<joint name="Revolute6" type="continuous">
   <origin xyz="0.0127 -0.154763 -0.027289" rpy="0 0 0"/>
   <parent link="link_6_1"/>
