Commit message: moveit config stuff dependant on it updated

File: robot_moveit_config/config/spotarm_assembly.ros2_control.xacro (robot description, xacro)
@@ -50,4 +50,11 @@
                 <state_interface name="velocity"/>
             </joint>
+            <joint name="gripper_right_finger_joint">
+                <command_interface name="position"/>
+                <state_interface name="position">
+                  <param name="initial_value">${initial_positions['gripper_right_finger_joint']}</param>
+                </state_interface>
+                <state_interface name="velocity"/>
+            </joint>
         </ros2_control>
     </xacro:macro>

File: spotarm_assembly_description/urdf/spotarm_assembly.ros2_control.xacro (robot description, xacro)
@@ -59,4 +59,11 @@
           <param name="default_velocity">0.2</param>
       </joint>
+      <joint name="gripper_right_finger_joint">
+          <command_interface name="position"/>
+          <state_interface name="position">
+            <param name="initial_value">0.0</param>
+          </state_interface>
+          <state_interface name="velocity"/>
+      </joint>
   </ros2_control>
 </robot>

File: spotarm_assembly_description/urdf/spotarm_assembly.urdf (robot description, URDF)
Before this commit: robot spotarm_assembly, 7 links, 6 joints
Links:
- added link gripper_left_finger, mass 0.05; collision box size=0.005 0.02 0.0192; visual box size=0.005 0.02 0.0192
- added link gripper_right_finger, mass 0.05; collision box size=0.005 0.02 0.0192; visual box size=0.005 0.02 0.0192
- link base_link: geometry collision mesh filename=file:///home/chungus/msd_robot_arm_2/install/spotarm_assemb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 scale=0.001 0.001 0.001; visual mesh filename=file:///home/chungus/msd_robot_arm_2/install/spotarm_assemb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 scale=0.001 0.001 0.001
- link gripper_1: geometry collision mesh filename=file:///home/chungus/msd_robot_arm_2/install/spotarm_assemb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 scale=0.001 0.001 0.001; visual mesh filename=file:///home/chungus/msd_robot_arm_2/install/spotarm_assemb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 scale=0.001 0.001 0.001
- link link_2_1: geometry collision mesh filename=file:///home/chungus/msd_robot_arm_2/install/spotarm_assemb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 scale=0.001 0.001 0.001; visual mesh filename=file:///home/chungus/msd_robot_arm_2/install/spotarm_assemb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 scale=0.001 0.001 0.001
- link link_3_1: geometry collision mesh filename=file:///home/chungus/msd_robot_arm_2/install/spotarm_assemb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 scale=0.001 0.001 0.001; visual mesh filename=file:///home/chungus/msd_robot_arm_2/install/spotarm_assemb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 scale=0.001 0.001 0.001
- link link_4_1: geometry collision mesh filename=file:///home/chungus/msd_robot_arm_2/install/spotarm_assemb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 scale=0.001 0.001 0.001; visual mesh filename=file:///home/chungus/msd_robot_arm_2/install/spotarm_assemb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 scale=0.001 0.001 0.001
- link link_5_1: geometry collision mesh filename=file:///home/chungus/msd_robot_arm_2/install/spotarm_assemb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 scale=0.001 0.001 0.001; visual mesh filename=file:///home/chungus/msd_robot_arm_2/install/spotarm_assemb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 scale=0.001 0.001 0.001
- link link_6_1: geometry collision mesh filename=file:///home/chungus/msd_robot_arm_2/install/spotarm_assemb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 scale=0.001 0.001 0.001; visual mesh filename=file:///home/chungus/msd_robot_arm_2/install/spotarm_assemb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 scale=0.001 0.001 0.001
Joints:
- added joint gripper_left_finger_joint: type prismatic, parent gripper_1, child gripper_left_finger, origin xyz=0.021 -0.0965 -0.0170 rpy=0.175 0 0, axis -1 0 0, limit lower=0.0 upper=0.0185 effort=10.0 velocity=0.02, mimic joint=gripper_right_finger_joint
- added joint gripper_right_finger_joint: type prismatic, parent gripper_1, child gripper_right_finger, origin xyz=-0.021 -0.0965 -0.0170 rpy=0.175 0 0, axis 1 0 0, limit lower=0.0 upper=0.0185 effort=10.0 velocity=0.02
- joint Revolute1: limit (none) -> lower=-0.436 upper=2.13 effort=30.0 velocity=1.0; type continuous -> revolute
- joint Revolute5: origin xyz=0.0705 -0.143933 0.0 rpy=0 0 0 -> xyz=0.0705 -0.143933 0.0 rpy=-0.175 0 0

File: spotarm_assembly_description/urdf/spotarm_assembly.xacro (robot description, xacro)
@@ -146,21 +146,80 @@
 </link>
 <link name="gripper_right_finger">
-  <visual>
-    <origin xyz="0 0 0" rpy="0 0 0"/>
-    <geometry>
-      <box size="0.005 0.02 0.0192"/>
-    </geometry>
-    <material name="silver"/>
-  </visual>
+  <inertial>
+    <origin xyz="0 0 0" rpy="0 0 0"/>
+    <mass value="0.05"/>
+    <inertia ixx="3.333333333333334e-05" iyy="1.3333333333333334e-05" izz="3.333333333333334e-05" ixy="0.0" iyz="0.0" ixz="0.0"/>
+  </inertial>
+  <visual>
+    <origin xyz="0 0 0" rpy="0 0 0"/>
+    <geometry>
+      <box size="0.005 0.02 0.0192"/>
+    </geometry>
+    <material name="silver"/>
+  </visual>
+  <collision>
+    <origin xyz="0 0 0" rpy="0 0 0"/>
+    <geometry>
+      <box size="0.005 0.02 0.0192"/>
+    </geometry>
+  </collision>
 </link>
 <link name="gripper_left_finger">
-  <visual>
-    <origin xyz="0 0 0" rpy="0 0 0"/>
-    <geometry>
-      <box size="0.005 0.02 0.0192"/>
-    </geometry>
-    <material name="silver"/>
-  </visual>
-</link>
+  <inertial>
+    <origin xyz="0 0 0" rpy="0 0 0"/>
+    <mass value="0.05"/>
+    <inertia ixx="3.333333333333334e-05" iyy="1.3333333333333334e-05" izz="3.333333333333334e-05" ixy="0.0" iyz="0.0" ixz="0.0"/>
+  </inertial>
+  <visual>
+    <origin xyz="0 0 0" rpy="0 0 0"/>
+    <geometry>
+      <box size="0.005 0.02 0.0192"/>
+    </geometry>
+    <material name="silver"/>
+  </visual>
+  <collision>
+    <origin xyz="0 0 0" rpy="0 0 0"/>
+    <geometry>
+      <box size="0.005 0.02 0.0192"/>
+    </geometry>
+  </collision>
+</link>
+<joint name="Revolute1" type="revolute">
+  <origin xyz="0.02835 -0.011972 0.033179" rpy="0 0 0"/>
+  <parent link="base_link"/>
+  <child link="link_2_1"/>
+  <axis xyz="-0.0 0.0 1.0"/>
+  <limit lower="-0.436" upper="2.13" effort="30.0" velocity="1.0"/>
+</joint>
+<joint name="Revolute2" type="continuous">
+  <origin xyz="0.046008 0.0 0.076206" rpy="0 0 0"/>
+  <parent link="link_2_1"/>
+  <child link="link_3_1"/>
+  <axis xyz="1.0 -0.0 -0.0"/>
+</joint>
+<joint name="Revolute3" type="continuous">
+  <origin xyz="-0.07256 -0.31369 0.0" rpy="0 0 0"/>
+  <parent link="link_3_1"/>
+  <child link="link_4_1"/>
+  <axis xyz="-1.0 0.0 0.0"/>
+</joint>
+<joint name="Revolute4" type="continuous">
+  <origin xyz="-0.012461 -0.2118 0.0" rpy="0 0 0"/>
+  <parent link="link_4_1"/>
+  <child link="link_5_1"/>
+  <axis xyz="-0.0 -1.0 0.0"/>
+</joint>
+<joint name="Revolute5" type="continuous">
+  <origin xyz="0.0705 -0.143933 0.0" rpy="-0.175 0 0"/>
+  <parent link="link_5_1"/>
+  <child link="link_6_1"/>
+  <axis xyz="1.0 -0.0 -0.0"/>
+</joint>
+<joint name="Revolute6" type="continuous">
+  <origin xyz="0.0127 -0.154763 -0.027289" rpy="0 0 0"/>
+  <parent link="link_6_1"/>
+  <child link="gripper_1"/>
+  <axis xyz="0.0 0.984808 0.173648"/>
+</joint>
 <joint name="gripper_right_finger_joint" type="prismatic">
   <parent link="gripper_1"/>
@@ -178,40 +237,3 @@
   <limit lower="0.0" upper="0.0185" effort="10.0" velocity="0.02"/>
 </joint>
-<joint name="Revolute1" type="revolute">
-  <origin xyz="0.02835 -0.011972 0.033179" rpy="0 0 0"/>
-  <parent link="base_link"/>
-  <child link="link_2_1"/>
-  <axis xyz="-0.0 0.0 1.0"/>
-  <limit lower="-0.436" upper="2.13" effort="30.0" velocity="1.0"/>
-</joint>
-<joint name="Revolute2" type="continuous">
-  <origin xyz="0.046008 0.0 0.076206" rpy="0 0 0"/>
-  <parent link="link_2_1"/>
-  <child link="link_3_1"/>
-  <axis xyz="1.0 -0.0 -0.0"/>
-</joint>
-<joint name="Revolute3" type="continuous">
-  <origin xyz="-0.07256 -0.31369 0.0" rpy="0 0 0"/>
-  <parent link="link_3_1"/>
-  <child link="link_4_1"/>
-  <axis xyz="-1.0 0.0 0.0"/>
-</joint>
-<joint name="Revolute4" type="continuous">
-  <origin xyz="-0.012461 -0.2118 0.0" rpy="0 0 0"/>
-  <parent link="link_4_1"/>
-  <child link="link_5_1"/>
-  <axis xyz="-0.0 -1.0 0.0"/>
-</joint>
-<joint name="Revolute5" type="continuous">
-  <origin xyz="0.0705 -0.143933 0.0" rpy="-0.175 0 0"/>
-  <parent link="link_5_1"/>
-  <child link="link_6_1"/>
-  <axis xyz="1.0 -0.0 -0.0"/>
-</joint>
-<joint name="Revolute6" type="continuous">
-  <origin xyz="0.0127 -0.154763 -0.027289" rpy="0 0 0"/>
-  <parent link="link_6_1"/>
-  <child link="gripper_1"/>
-  <axis xyz="0.0 0.984808 0.173648"/>
-</joint>
 </robot>

Commit message: remove fingers

File: robot_moveit_config/config/spotarm_assembly.ros2_control.xacro (robot description, xacro)
@@ -50,11 +50,4 @@
                 <state_interface name="velocity"/>
             </joint>
-            <joint name="gripper_right_finger_joint">
-                <command_interface name="position"/>
-                <state_interface name="position">
-                  <param name="initial_value">${initial_positions['gripper_right_finger_joint']}</param>
-                </state_interface>
-                <state_interface name="velocity"/>
-            </joint>
         </ros2_control>
     </xacro:macro>

File: spotarm_assembly_description/urdf/spotarm_assembly.ros2_control.xacro (robot description, xacro)
@@ -59,11 +59,4 @@
           <param name="default_velocity">0.2</param>
       </joint>
-      <joint name="gripper_right_finger_joint">
-          <command_interface name="position"/>
-          <state_interface name="position">
-            <param name="initial_value">0.0</param>
-          </state_interface>
-          <state_interface name="velocity"/>
-      </joint>
   </ros2_control>
 </robot>

File: spotarm_assembly_description/urdf/spotarm_assembly.xacro (robot description, xacro)
@@ -145,5 +145,5 @@
   </collision>
 </link>
-<link name="gripper_right_finger">
+<!-- <link name="gripper_right_finger">
   <inertial>
     <origin xyz="0 0 0" rpy="0 0 0"/>
@@ -184,5 +184,5 @@
     </geometry>
   </collision>
-</link>
+</link> -->
 <joint name="Revolute1" type="revolute">
   <origin xyz="0.02835 -0.011972 0.033179" rpy="0 0 0"/>
@@ -222,5 +222,5 @@
   <axis xyz="0.0 0.984808 0.173648"/>
 </joint>
-<joint name="gripper_right_finger_joint" type="prismatic">
+<!-- <joint name="gripper_right_finger_joint" type="prismatic">
   <parent link="gripper_1"/>
   <child link="gripper_right_finger"/>
@@ -236,4 +236,4 @@
   <mimic joint="gripper_right_finger_joint"/>
   <limit lower="0.0" upper="0.0185" effort="10.0" velocity="0.02"/>
-</joint>
+</joint> -->
 </robot>
